File: pcb_design_1/pcb/5v_in.kicad_sch (KiCad schematic)
At the start: 3 parts, among them U3 LM7812_TO220

Commit message: Add OLED Display and power switch, rename battery input
Added new OLED Display schematic sheet with I2C connector (J14) and pinout. Integrated OLED display connections (VCC, GND, SDA, SCL) into main PCB. Added power switch (SW1) between battery input and power supply. Renamed battery input signal from 'battery_in' to 'battery_in_1' throughout 5V input and power supply sheets. Updated component designators and repositioned schematic sheets for improved layout organization.
Connections:
- net battery_in renamed battery_in_1
Changed lines of the file:
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@@
 		)
 	)
-	(hierarchical_label "battery_in"
+	(hierarchical_label "battery_in_1"
 		(shape input)
 		(at 115.57 73.66 180)
