File: pcb_design_1/pcb/ESP32.kicad_sch (KiCad schematic)
At the start: 7 parts, among them J10 Conn_01x02_Pin, J8 Conn_01x03_Pin, U5 ESP32-WROOM-32

Commit message: Add TOF sensor sheet and move I2C resistors
- Created new Sensors_TOF schematic sheet for Time-of-Flight sensor with I2C interface
- Moved I2C pull-up resistors (R8, R9, 2k ohm) from PCF8574 to ESP32 sheet
- Added hierarchical labels (SDA, SCL, 3.3v) to ESP32 sheet for I2C connectivity
- Added TOF sensor connector (J7) with 6-pin socket connection
- Updated project designators in pcb.kicad_pro
Parts:
- added R8, R9: 2k, symbol Device:R
Connections:
- new net 3.3v: R8.1, R9.1
- new net SCL: R9.2
- new net SDA: R8.2

Commit message: Update KiCad sheet wiring
Adjust schematic hierarchy and net connections across the PCB project, including ESP32, TCA9548A, OLED, sensors, switches, and indication sheets. Adds R1 and updates sheet pin labels, wire placement, and project designator metadata to match the revised net naming and connectivity.
Connections:
- net CLK is gone; now on net SCL: U5.20 (SCK/CLK)
- net SDO is gone; now on net SDA: U5.21 (SDO/SD0)
- net TCA9548A_RST: now reaches U5.10 (IO25)
Changed lines of the file:
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@@
 	(wire
 		(pts
+			(xy 149.86 105.41) (xy 165.1 105.41)
+		)
+		(stroke
+			(width 0)
+			(type default)
+		)
+	)
+	(wire
+		(pts
 			(xy 177.8 24.13) (xy 185.42 24.13)
 		)
@@
 		)
 	)
+	(label "SDA"
+		(at 105.41 92.71 180)
+		(effects
+			(font
+				(size 1.27 1.27)
+			)
+			(justify right bottom)
+		)
+	)
 	(label "RXDO"
 		(at 258.572 74.93 180)
@@
 		)
 	)
+	(label "SCL"
+		(at 105.41 102.87 180)
+		(effects
+			(font
+				(size 1.27 1.27)
+			)
+			(justify right bottom)
+		)
+	)
 	(label "CAN_TXD"
 		(at 149.86 72.39 0)
@@
 		)
 	)
-	(hierarchical_label "SDO"
+	(hierarchical_label "TCA9548A_RST"
 		(shape input)
-		(at 105.41 92.71 180)
+		(at 165.1 105.41 0)
 		(effects
 			(font
 				(size 1.27 1.27)
 			)
-			(justify right)
+			(justify left)
 		)
 	)
@@
 		)
 	)
-	(hierarchical_label "CLK"
-		(shape input)
-		(at 105.41 102.87 180)
-		(effects
-			(font
-				(size 1.27 1.27)
-			)
-			(justify right)
-		)
-	)
