File: pcb_design_1/pcb/OLED_Display.kicad_sch (KiCad schematic)
At the start: 1 part, among them J14 Conn_01x04_Socket

Commit message: improved the designed
improved the designed
Other:
- moved on the sheet: J14
Changed lines of the file:
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@@
 	(wire
 		(pts
-			(xy 91.44 96.52) (xy 91.44 77.47)
+			(xy 105.41 96.52) (xy 105.41 77.47)
 		)
 		(stroke
@@
 	(wire
 		(pts
-			(xy 88.9 96.52) (xy 88.9 77.47)
+			(xy 102.87 96.52) (xy 102.87 77.47)
 		)
 		(stroke
@@
 	(wire
 		(pts
-			(xy 96.52 96.52) (xy 96.52 77.47)
+			(xy 110.49 96.52) (xy 110.49 77.47)
 		)
 		(stroke
@@
 	(wire
 		(pts
-			(xy 93.98 96.52) (xy 93.98 77.47)
+			(xy 99.06 77.47) (xy 102.87 77.47)
+		)
+		(stroke
+			(width 0)
+			(type default)
+		)
+	)
+	(wire
+		(pts
+			(xy 107.95 96.52) (xy 107.95 77.47)
 		)
 		(stroke
@@
 	(hierarchical_label "VCC"
 		(shape input)
-		(at 91.44 77.47 90)
+		(at 105.41 77.47 90)
 		(effects
 			(font
@@
 	(hierarchical_label "SDA"
 		(shape input)
-		(at 96.52 77.47 90)
+		(at 110.49 77.47 90)
 		(effects
 			(font
@@
 	(hierarchical_label "SCL"
 		(shape input)
-		(at 93.98 77.47 90)
+		(at 107.95 77.47 90)
 		(effects
 			(font
@@
 		)
 	)
-	(hierarchical_label "GND"
-		(shape input)
-		(at 88.9 77.47 90)
-		(effects
-			(font
-				(size 1.27 1.27)
-			)
-			(justify left)
+	(symbol
+		(lib_id "power:GND")
+		(at 99.06 77.47 0)
+		(unit 1)
+		(body_style 1)
+		(exclude_from_sim no)
+		(in_bom yes)
+		(on_board yes)
+		(in_pos_files yes)
+		(dnp no)
+		(fields_autoplaced yes)
+		(property "Reference" "#PWR029"
+			(at 99.06 83.82 0)
+			(hide yes)
+			(show_name no)
+			(do_not_autoplace no)
+			(effects
+				(font
+					(size 1.27 1.27)
+				)
+			)
+		)
+		(property "Value" "GND"
+			(at 99.06 82.55 0)
+			(show_name no)
+			(do_not_autoplace no)
+			(effects
+				(font
+					(size 1.27 1.27)
+				)
+			)
+		)
+		(property "Footprint" ""
+			(at 99.06 77.47 0)
+			(hide yes)
+			(show_name no)
+			(do_not_autoplace no)
+			(effects
+				(font
+					(size 1.27 1.27)
+				)
+			)
+		)
+		(property "Datasheet" ""
+			(at 99.06 77.47 0)
+			(hide yes)
+			(show_name no)
+			(do_not_autoplace no)
+			(effects
+				(font
+					(size 1.27 1.27)
+				)
+			)
+		)
+		(property "Description" "Power symbol creates a global label with name \"GND\" , ground"
+			(at 99.06 77.47 0)
+			(hide yes)
+			(show_name no)
+			(do_not_autoplace no)
+			(effects
+				(font
+					(size 1.27 1.27)
+				)
+			)
+		)
+		(pin "1"
+		)
+		(instances
+			(project "pcb"
+				(path "/641f7b51-eb90-47ac-8b04-a4718aaaca74/170bd367-671e-47a1-a124-6effc20b5547"
+					(reference "#PWR029")
+					(unit 1)
+				)
+			)
 		)
 	)
 	(symbol
 		(lib_id "Connector:Conn_01x04_Socket")
-		(at 93.98 101.6 270)
+		(at 107.95 101.6 270)
 		(unit 1)
 		(body_style 1)
@@
 		(fields_autoplaced yes)
 		(property "Reference" "J14"
-			(at 83.82 100.965 0)
+			(at 97.79 100.965 0)
 			(show_name no)
 			(do_not_autoplace no)
@@
 		)
 		(property "Value" "Conn_01x04_Socket"
-			(at 86.36 100.965 0)
+			(at 100.33 100.965 0)
 			(show_name no)
 			(do_not_autoplace no)
@@
 		)
 		(property "Footprint" ""
-			(at 93.98 101.6 0)
+			(at 107.95 101.6 0)
 			(hide yes)
 			(show_name no)
@@
 		)
 		(property "Datasheet" ""
-			(at 93.98 101.6 0)
+			(at 107.95 101.6 0)
 			(hide yes)
 			(show_name no)
@@
 		)
 		(property "Description" "Generic connector, single row, 01x04, script generated"
-			(at 93.98 101.6 0)
+			(at 107.95 101.6 0)
 			(hide yes)
 			(show_name no)
