File: pcb_design_1/pcb/Sensors_TOF.kicad_sch (KiCad schematic)
At the start: 5 parts, among them J11 Conn_01x06_Socket, J12 Conn_01x06_Socket, J13 Conn_01x06_Socket, J7 Conn_01x06_Socket, J9 Conn_01x06_Socket

Commit message: improved the designed
improved the designed
Connections:
- removed net SCL: J11.4 (Pin_4), J12.4 (Pin_4), J13.4 (Pin_4), J7.4 (Pin_4), J9.4 (Pin_4)
- removed net SDA: J11.3 (Pin_3), J12.3 (Pin_3), J13.3 (Pin_3), J7.3 (Pin_3), J9.3 (Pin_3)
- new net SCL_1: J7.4 (Pin_4)
- new net SCL_2: J9.4 (Pin_4)
- new net SCL_3: J11.4 (Pin_4)
- new net SCL_4: J12.4 (Pin_4)
- new net SCL_5: J13.4 (Pin_4)
- new net SDA_1: J7.3 (Pin_3)
- new net SDA_2: J9.3 (Pin_3)
- new net SDA_3: J11.3 (Pin_3)
- new net SDA_4: J12.3 (Pin_3)
- new net SDA_5: J13.3 (Pin_3)
